File: hardware/pcb/display-board/display-board.kicad_sch (KiCad schematic)
At the start: 46 parts, among them J1 Conn_01x01_Socket, J2 Conn_01x01_Socket, J3 Conn_01x01_Socket, J4 Conn_01x01_Socket, J5 Conn_01x01_Socket, J6 Conn_01x01_Socket, Q1 AO3400A, Q2 AO3401A, Q3 AO3400A, Q4 AO3401A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

Commit message: Added main board to the hw folder, some 3d models for the inner structure and the code itself
Parts:
- added C1: C, Capacitor_SMD:C_0603_1608Metric_Pad1.08x0.95mm_HandSolder, symbol Device:C
- added C2, C3: 0.1uF, Capacitor_SMD:C_0805_2012Metric_Pad1.18x1.45mm_HandSolder, symbol Device:C
- added R11, R13: 1k, Resistor_SMD:R_0603_1608Metric_Pad0.98x0.95mm_HandSolder, symbol Device:R
- added R12, R14: 100k, Resistor_SMD:R_0603_1608Metric_Pad0.98x0.95mm_HandSolder, symbol Device:R
Connections:
- net BUZZER: now also PWR1.3 (Pin_3), PWR2.3 (Pin_3), PWR3.3 (Pin_3), PWR4.3 (Pin_3)
- net CTRL: now also DD1.2 (Pin_2), DD2.2 (Pin_2); no longer PWR1.3 (Pin_3), PWR2.3 (Pin_3), PWR3.3 (Pin_3), PWR4.3 (Pin_3)
- net GND: now also C1.2, C2.2, C3.2
- net LDO: now also R12.1, R14.1
- net SW1: now also C3.1, R13.2, R14.2; no longer SW1.1
- net SW2: now also C2.1, R11.2, R12.2; no longer SW2.2
- net VCC: now also U1.26 (DCPRG), C1.1
- removed net DCPRG: DD1.2 (Pin_2), DD2.2 (Pin_2), U1.26 (DCPRG)
- new net: R13.1, SW1.1
- new net: R11.1, SW2.2
Other:
- moved on the sheet: BZ1, D1, PWR_S1, Q7, R10, R8, R9, SW1, SW2
