File: hardware/pcb/main-board-v2/main-board.kicad_sch (KiCad schematic)
At the start: 136 parts, among them J1 USB_C_Receptacle_USB2.0_16P, P11 TestPoint_Alt, P12 TestPoint_Alt, P13 TestPoint_Alt, P46 TestPoint_Alt, Q1 AO3401A, Q2 AO3401A, Q3 AO3400A, Q4 AO3401A, Q5 AO3401A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

Commit message: Added project basis, software, hardware and 3d models
Connections:
- net -BATT: no longer BAT1.1 (Pin_1), R35.1, U7.3 (BAT-)
- net GND: now also R35.1, U7.3 (BAT-); no longer C18.2, U7.1 (GND)
- new net: BAT1.1 (Pin_1), C18.2, U7.1 (GND)
Other:
- note added: "B-"
- note added: "don't forget to route ldo_ctrl"
- moved on the sheet: BAT1, R35, U7
Changed lines of the file:
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@@
 	)
 	(junction
-		(at 401.32 72.39)
+		(at 106.68 165.1)
 		(diameter 0)
 		(color 0 0 0 0)
 	)
 	(junction
-		(at 106.68 165.1)
+		(at 214.63 -45.72)
 		(diameter 0)
 		(color 0 0 0 0)
 	)
 	(junction
-		(at 214.63 -45.72)
+		(at 175.26 33.02)
 		(diameter 0)
 		(color 0 0 0 0)
 	)
 	(junction
-		(at 175.26 33.02)
+		(at 447.04 60.96)
 		(diameter 0)
 		(color 0 0 0 0)
@@
 	)
 	(junction
-		(at 448.31 45.72)
-		(diameter 0)
-		(color 0 0 0 0)
-	)
-	(junction
 		(at 430.53 134.62)
 		(diameter 0)
@@
 	)
 	(junction
-		(at 443.23 60.96)
-		(diameter 0)
-		(color 0 0 0 0)
-	)
-	(junction
 		(at 256.54 -30.48)
 		(diameter 0)
@@
 	)
 	(junction
+		(at 408.94 72.39)
+		(diameter 0)
+		(color 0 0 0 0)
+	)
+	(junction
 		(at 430.53 124.46)
 		(diameter 0)
@@
 	(wire
 		(pts
+			(xy 447.04 64.77) (xy 447.04 60.96)
+		)
+		(stroke
+			(width 0)
+			(type default)
+		)
+	)
+	(wire
+		(pts
 			(xy -27.94 57.15) (xy -33.02 57.15)
 		)
@@
 	(wire
 		(pts
-			(xy 420.37 45.72) (xy 420.37 43.18)
+			(xy 408.94 43.18) (xy 408.94 72.39)
 		)
 		(stroke
@@
 	(wire
 		(pts
-			(xy 448.31 45.72) (xy 420.37 45.72)
-		)
-		(stroke
-			(width 0)
-			(type default)
-		)
-	)
-	(wire
-		(pts
 			(xy 57.15 52.07) (xy 57.15 53.34)
 		)
@@
 	(wire
 		(pts
-			(xy 401.32 72.39) (xy 401.32 74.93)
-		)
-		(stroke
-			(width 0)
-			(type default)
-		)
-	)
-	(wire
-		(pts
 			(xy -78.74 54.61) (xy -83.82 54.61)
 		)
@@
 	(wire
 		(pts
-			(xy 389.89 45.72) (xy 417.83 45.72)
+			(xy 389.89 45.72) (xy 406.4 45.72)
 		)
 		(stroke
@@
 	(wire
 		(pts
-			(xy 408.94 60.96) (xy 408.94 72.39)
+			(xy 414.02 60.96) (xy 414.02 72.39)
 		)
 		(stroke
@@
 	(wire
 		(pts
-			(xy 430.53 60.96) (xy 443.23 60.96)
-		)
-		(stroke
-			(width 0)
-			(type default)
-		)
-	)
-	(wire
-		(pts
 			(xy 160.02 46.99) (xy 163.83 46.99)
 		)
@@
 	(wire
 		(pts
-			(xy 401.32 58.42) (xy 408.94 58.42)
+			(xy 401.32 58.42) (xy 414.02 58.42)
 		)
 		(stroke
@@
 	(wire
 		(pts
-			(xy 430.53 58.42) (xy 435.61 58.42)
+			(xy 435.61 58.42) (xy 439.42 58.42)
 		)
 		(stroke
@@
 	(wire
 		(pts
+			(xy 408.94 72.39) (xy 401.32 72.39)
+		)
+		(stroke
+			(width 0)
+			(type default)
+		)
+	)
+	(wire
+		(pts
 			(xy 316.23 54.61) (xy 316.23 58.42)
 		)
@@
 	(wire
 		(pts
-			(xy 443.23 60.96) (xy 443.23 58.42)
+			(xy 447.04 60.96) (xy 447.04 58.42)
 		)
 		(stroke
@@
 	(wire
 		(pts
-			(xy 448.31 60.96) (xy 448.31 45.72)
+			(xy 435.61 60.96) (xy 447.04 60.96)
 		)
 		(stroke
@@
 	(wire
 		(pts
-			(xy 408.94 72.39) (xy 401.32 72.39)
+			(xy 414.02 72.39) (xy 408.94 72.39)
 		)
 		(stroke
@@
 	(wire
 		(pts
-			(xy 417.83 45.72) (xy 417.83 43.18)
+			(xy 406.4 45.72) (xy 406.4 43.18)
 		)
 		(stroke
@@
 	(wire
 		(pts
-			(xy 448.31 43.18) (xy 448.31 45.72)
-		)
-		(stroke
-			(width 0)
-			(type default)
-		)
-	)
-	(wire
-		(pts
 			(xy 55.88 40.64) (xy 72.39 40.64)
 		)
@@
 	(wire
 		(pts
-			(xy 443.23 60.96) (xy 448.31 60.96)
-		)
-		(stroke
-			(width 0)
-			(type default)
-		)
-	)
-	(wire
-		(pts
 			(xy -78.74 49.53) (xy -83.82 49.53)
 		)
@@
 		)
 	)
+	(text "don't forget to route ldo_ctrl"
+		(exclude_from_sim no)
+		(at 107.442 111.76 0)
+		(effects
+			(font
+				(size 1.27 1.27)
+			)
+		)
+	)
 	(text "Connectors"
 		(exclude_from_sim no)
@@
 		)
 	)
+	(text "B-"
+		(exclude_from_sim no)
+		(at 410.972 45.212 0)
+		(effects
+			(font
+				(size 1.27 1.27)
+			)
+		)
+	)
 	(text "Regulator"
 		(exclude_from_sim no)
@@
 	(symbol
 		(lib_id "power:GND")
-		(at 401.32 74.93 0)
+		(at 447.04 64.77 0)
 		(unit 1)
 		(exclude_from_sim no)
@@
 		(fields_autoplaced yes)
 		(property "Reference" "#PWR052"
-			(at 401.32 81.28 0)
+			(at 447.04 71.12 0)
 			(effects
 				(font
@@
 		)
 		(property "Value" "GND"
-			(at 401.32 80.01 0)
+			(at 447.04 69.85 0)
 			(effects
 				(font
@@
 		)
 		(property "Footprint" ""
-			(at 401.32 74.93 0)
+			(at 447.04 64.77 0)
 			(effects
 				(font
@@
 		)
 		(property "Datasheet" ""
-			(at 401.32 74.93 0)
+			(at 447.04 64.77 0)
 			(effects
 				(font
@@
 		)
 		(property "Description" "Power symbol creates a global label with name \"GND\" , ground"
-			(at 401.32 74.93 0)
+			(at 447.04 64.77 0)
 			(effects
 				(font
@@
 	(symbol
 		(lib_id "Power_Management:FS312MH")
-		(at 411.48 64.77 0)
+		(at 416.56 64.77 0)
 		(unit 1)
 		(exclude_from_sim no)
@@
 		(fields_autoplaced yes)
 		(property "Reference" "U7"
-			(at 419.735 50.8 0)
+			(at 424.815 50.8 0)
 			(effects
 				(font
@@
 		)
 		(property "Value" "FS312MH"
-			(at 419.735 53.34 0)
+			(at 424.815 53.34 0)
 			(effects
 				(font
@@
 		)
 		(property "Footprint" "Package_TO_SOT_SMD:SOT-23-6_Handsoldering"
-			(at 416.56 72.39 0)
+			(at 421.64 72.39 0)
 			(effects
 				(font
@@
 		)
 		(property "Datasheet" ""
-			(at 411.48 64.77 0)
+			(at 416.56 64.77 0)
 			(effects
 				(font
@@
 		)
 		(property "Description" ""
-			(at 411.48 64.77 0)
+			(at 416.56 64.77 0)
 			(effects
 				(font
@@
 	(symbol
 		(lib_id "Connector:Conn_01x02_Pin")
-		(at 420.37 38.1 270)
+		(at 408.94 38.1 270)
 		(unit 1)
 		(exclude_from_sim no)
@@
 		(fields_autoplaced yes)
 		(property "Reference" "BAT1"
-			(at 421.64 37.4649 90)
+			(at 410.21 37.4649 90)
 			(effects
 				(font
@@
 		)
 		(property "Value" "Conn_01x02_Pin"
-			(at 421.64 40.0049 90)
+			(at 410.21 40.0049 90)
 			(effects
 				(font
@@
 		)
 		(property "Footprint" "Connector_JST:JST_XH_B2B-XH-A_1x02_P2.50mm_Vertical"
-			(at 420.37 38.1 0)
+			(at 408.94 38.1 0)
 			(effects
 				(font
@@
 		)
 		(property "Datasheet" "~"
-			(at 420.37 38.1 0)
+			(at 408.94 38.1 0)
 			(effects
 				(font
@@
 		)
 		(property "Description" "Generic connector, single row, 01x02, script generated"
-			(at 420.37 38.1 0)
+			(at 408.94 38.1 0)
 			(effects
 				(font
@@
 	(symbol
 		(lib_id "Device:R")
-		(at 439.42 58.42 270)
+		(at 443.23 58.42 270)
 		(unit 1)
 		(exclude_from_sim no)
@@
 		(fields_autoplaced yes)
 		(property "Reference" "R35"
-			(at 439.42 52.07 90)
+			(at 443.23 52.07 90)
 			(effects
 				(font
@@
 		)
 		(property "Value" "2K"
-			(at 439.42 54.61 90)
+			(at 443.23 54.61 90)
 			(effects
 				(font
@@
 		)
 		(property "Footprint" "Resistor_SMD:R_0603_1608Metric_Pad0.98x0.95mm_HandSolder"
-			(at 439.42 56.642 90)
+			(at 443.23 56.642 90)
 			(effects
 				(font
@@
 		)
 		(property "Datasheet" "~"
-			(at 439.42 58.42 0)
+			(at 443.23 58.42 0)
 			(effects
 				(font
@@
 		)
 		(property "Description" "Resistor"
-			(at 439.42 58.42 0)
+			(at 443.23 58.42 0)
 			(effects
 				(font
@@
 					(unit 1)
 				)
-			)
-		)
-	)
-	(symbol
-		(lib_id "power:-BATT")
-		(at 448.31 43.18 0)
-		(unit 1)
-		(exclude_from_sim no)
-		(in_bom yes)
-		(on_board yes)
-		(dnp no)
-		(fields_autoplaced yes)
-		(property "Reference" "#PWR057"
-			(at 448.31 46.99 0)
-			(effects
-				(font
-					(size 1.27 1.27)
-				)
-				(hide yes)
-			)
-		)
-		(property "Value" "-BATT"
-			(at 448.31 38.1 0)
-			(effects
-				(font
-					(size 1.27 1.27)
-				)
-			)
-		)
-		(property "Footprint" ""
-			(at 448.31 43.18 0)
-			(effects
-				(font
-					(size 1.27 1.27)
-				)
-				(hide yes)
-			)
-		)
-		(property "Datasheet" ""
-			(at 448.31 43.18 0)
-			(effects
-				(font
-					(size 1.27 1.27)
-				)
-				(hide yes)
-			)
-		)
-		(property "Description" "Power symbol creates a global label with name \"-BATT\""
-			(at 448.31 43.18 0)
-			(effects
-				(font
-					(size 1.27 1.27)
-				)
-				(hide yes)
-			)
-		)
-		(pin "1"
-		)
-		(instances
-			(project "main-board"
-				(path "/419474dc-89fd-407d-8968-c566cf752eb0"
-					(reference "#PWR057")
-					(unit 1)
-				)

Commit message: renamed some funcs/vars from camelCase to snake_case, added padel, moved initTasks to the end
Parts:
- removed C10, C11, C12, C9: 0.1uF, Capacitor_SMD:C_0805_2012Metric_Pad1.18x1.45mm_HandSolder, symbol Device:C
- removed R20, R23: 1k, Capacitor_SMD:C_0603_1608Metric_Pad1.08x0.95mm_HandSolder, symbol Device:R
- removed R21, R22: 4.7k, Capacitor_SMD:C_0603_1608Metric_Pad1.08x0.95mm_HandSolder, symbol Device:R
- removed U3, U4: BH1750FVI-TR, BH1750FVI-TR:XDCR_BH1750FVI-TR, symbol BH1750FVI-TR:BH1750FVI-TR
Connections:
- net -BATT: now also BAT1.1 (Pin_1), C18.2, U7.1 (GND)
Other:
- note removed: "B-"
- note removed: "Light Sensors"
