File: hardware/pcb/v2.0/main-board/main-board.kicad_sch (KiCad schematic)
At the start: 126 parts, among them J1 USB_C_Receptacle_USB2.0_16P, P11 TestPoint_Alt, P12 TestPoint_Alt, P13 TestPoint_Alt, P46 TestPoint_Alt, Q1 AO3401A, Q2 AO3401A, Q3 AO3400A, Q4 AO3401A, Q5 AO3401A, Q6 AO3401A, Q7 AO3400A, Q8 AO3401A, Q9 AO3401A, U1 TL431DBZ, U2 ESP32-S3-WROOM-1, U5 AP2112K-3.3, U6 TP4056, U7 FS312MH, U8 ESP32-S2-WROVER-I

Commit message: updated v2 main board
removed redundant parts (light sensor that was never used and many jumpers)
added an analog switch to detect and route mosi signal to display board
fixed batt circuit
replaced single row connectors by one double each side (mirrored)
Parts:
- removed AB_1, AB_2, AB_3, ALT_A1, ALT_B1, SW_1, SW_2: SolderJumper_3_Open, Jumper:SolderJumper-3_P1.3mm_Open_RoundedPad1.0x1.5mm_NumberLabels, symbol Jumper:SolderJumper_3_Open
- removed CA1, CA2, CA3, CA4, PWR1, PWR2, PWR3, PWR4: Conn_01x04_Pin, Connector_PinHeader_1.27mm:PinHeader_1x04_P1.27mm_Vertical, symbol Connector:Conn_01x04_Pin
- removed D2: BAT20JFILM, BAT20JFILM:SOD-323, symbol BAT20JFILM:BAT20JFILM
- removed D4, D5: LED, LED_SMD:LED_0603_1608Metric_Pad1.05x0.95mm_HandSolder, symbol Device:LED
- removed D9: BAT20J, BAT20JFILM:SOD-323, symbol BAT20JFILM:BAT20JFILM
- removed DD1, DD2, DD3, DD4: Conn_01x10_Pin, Connector_PinHeader_1.27mm:PinHeader_1x10_P1.27mm_Vertical, symbol Connector:Conn_01x10_Pin
- removed Q1, Q2: AO3401A, Package_TO_SOT_SMD:SOT-23, symbol Transistor_FET:AO3401A
- removed R15, R16: 2.2K, Resistor_SMD:R_0603_1608Metric_Pad0.98x0.95mm_HandSolder, symbol Device:R
- removed R34: 1M, Resistor_SMD:R_0603_1608Metric_Pad0.98x0.95mm_HandSolder, symbol Device:R
- removed SW_C1, SW_C2, SW_C3, SW_C4: Conn_01x03_Pin, Connector_PinHeader_1.27mm:PinHeader_1x03_P1.27mm_Vertical, symbol Connector:Conn_01x03_Pin
- removed U1: TL431DBZ, Package_TO_SOT_SMD:SOT-23, symbol Reference_Voltage:TL431DBZ
- removed U8: ESP32-S2-WROVER-I, RF_Module:ESP32-S2-WROVER, symbol RF_Module:ESP32-S2-WROVER-I
- added C10: 2.2uF, Capacitor_SMD:C_0805_2012Metric_Pad1.18x1.45mm_HandSolder, symbol Device:C
- added C11: 10uF, Capacitor_SMD:C_0805_2012Metric_Pad1.18x1.45mm_HandSolder, symbol Device:C
- added C12, C7, C8: 0.1uF, Capacitor_SMD:C_0805_2012Metric_Pad1.18x1.45mm_HandSolder, symbol Device:C
- added C9: 10nF, Capacitor_SMD:C_0805_2012Metric_Pad1.18x1.45mm_HandSolder, symbol Device:C
- added D2, D9: LED, LED_SMD:LED_0603_1608Metric_Pad1.05x0.95mm_HandSolder, symbol Device:LED
- added J2, J3: Conn_02x12_Odd_Even, symbol Connector_Generic:Conn_02x12_Odd_Even
- added R20: 300, symbol Device:R
- added U1: 74LVC1G3157, symbol 74xGxx:74LVC1G3157
- added U3: DRV8833PWP, Package_SO:HTSSOP-16-1EP_4.4x5mm_P0.65mm_EP3.4x5mm_Mask2.46x2.31mm_ThermalVias, symbol Driver_Motor:DRV8833PWP
- C6: value 0.1uF -> 1nF; footprint Capacitor_SMD:C_0805_2012Metric_Pad1.18x1.45mm_HandSolder -> (none)
- D1: value BAT20JFILM -> BAT20J
- R10: value R -> 10k; footprint Capacitor_SMD:C_0603_1608Metric_Pad1.08x0.95mm_HandSolder -> Resistor_SMD:R_0603_1608Metric_Pad0.98x0.95mm_HandSolder
- R12: value 1M -> 2.2K
- R13: value R -> 2.2K; footprint Capacitor_SMD:C_0603_1608Metric_Pad1.08x0.95mm_HandSolder -> Resistor_SMD:R_0603_1608Metric_Pad0.98x0.95mm_HandSolder
- R14: value R -> 300; footprint Capacitor_SMD:C_0603_1608Metric_Pad1.08x0.95mm_HandSolder -> (none)
- R24, R25, R28, R30, R32, R33: value 1M -> 100k
- R3, R4: value R -> 1M
- R6: value 10k -> 56k
Connections:
- net +BATT: now also Q6.2 (S), R3.1; no longer Q6.3 (D), R6.1
- net -BATT: now also R35.1, U7.3 (BAT-); no longer C18.2, U7.1 (GND)
- net 1V: no longer C6.1, R13.2, R14.2, U2.39 (GPIO1/TOUCH1/ADC1_CH0)
- net 2.5V: no longer R10.1, R13.1
- net ADC_BAT_V: no longer R3.2, R4.1
- net BLANK: now also U2.9 (GPIO16/U0CTS/ADC2_CH5/XTAL_32K_N), J2.18 (Pin_18), J3.18 (Pin_18)
- net CTRL: now also U2.31 (GPIO38/FSPIWP/SUBSPIWP)
- net GND: now also C18.2, C3.1, R12.2, R13.1, U7.1 (GND), C10.1, C11.1, C12.1, C8.1, J2.10 (Pin_10), J2.15 (Pin_15), J2.16 (Pin_16), J2.22 (Pin_22), J2.23 (Pin_23), J2.5 (Pin_5), J2.6 (Pin_6), J3.10 (Pin_10), J3.15 (Pin_15), J3.16 (Pin_16), J3.22 (Pin_22), J3.23 (Pin_23), J3.5 (Pin_5), J3.6 (Pin_6), U1.2 (GND), U3.13 (GND), U3.17 (GND), U3.3 (AISEN), U3.6 (BISEN); no longer R14.1, R35.1, U7.3 (BAT-)
- net GSCLK: now also U2.11 (GPIO18/U1RXD/ADC2_CH7/CLK_OUT3), J2.24 (Pin_24), J3.24 (Pin_24)
- net LDO_CTRL: now also R10.2, C8.2, J2.3 (Pin_3), J2.4 (Pin_4), J3.3 (Pin_3), J3.4 (Pin_4), U1.5 (VCC), U3.1 (~{SLEEP})
- net LDO_CTRL_EN: now also U2.12 (GPIO8/TOUCH8/ADC1_CH7/SUBSPICS1)
- net LDO_LATCH: now also U2.7 (GPIO7/TOUCH7/ADC1_CH6)
- net MOSI(SIN): now also J2.20 (Pin_20), U1.1
- net SCLK: now also J2.21 (Pin_21), J3.21 (Pin_21)
- net SIN_B: now also J3.20 (Pin_20), U1.4
- net SOUT_A: now also J2.17 (Pin_17), U1.3
- net SOUT_B: now also J3.17 (Pin_17)
- net SW1: now also D1.C, J2.11 (Pin_11), J3.11 (Pin_11)
- net SW2: now also J2.12 (Pin_12), J3.12 (Pin_12); no longer D1.C
- net VBUS: now also R6.1; no longer R30.1
- net VCC: now also Q6.3 (D), C7.1; no longer Q6.2 (S), R12.1
- net VCC_CTRL: now also C11.2, C12.2, C9.2, J2.1 (Pin_1), J2.2 (Pin_2), J3.1 (Pin_1), J3.2 (Pin_2), U3.12 (VM)
- net VCC_CTRL_EN: now also U2.17 (GPIO9/TOUCH9/ADC1_CH8/FSPIHD/SUBSPIHD)
- net XLAT: now also U2.10 (GPIO17/U1TXD/ADC2_CH6), J2.19 (Pin_19), J3.19 (Pin_19)
- net at D8.A, Q7.3 (D), Q8.1 (G)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: now also C7.2
- net ADC_BAT: now reaches C3.2
- net ADC_BAT: now also R3.2, R4.1; no longer R6.2
- net at U2.16 (GPIO46): now also D9.2 (A)
- net GPIO_10: now reaches U2.18 (GPIO10/TOUCH10/ADC1_CH9/FSPICS0/FSPIIO4/SUBSPICS0)
- net GPIO14: now reaches U2.22 (GPIO14/TOUCH14/ADC2_CH3/FSPIWP/FSPIDQS/SUBSPIWP)
- net GPIO_21: now reaches U2.23 (GPIO21)
- net BZ_B_1: now reaches U2.24 (GPIO47/SPICLK_P/SUBSPICLK_P_DIFF)
- net BZ_B_1: now also U3.9 (BIN1)
- net BZ_B_2: now reaches U2.25 (GPIO48/SPICLK_N/SUBSPICLK_N_DIFF)
- net BZ_B_2: now also U3.10 (BIN2)
- net at U2.26 (GPIO45): now also D2.2 (A)
- net SLOT_A_DET: now reaches U2.28 (SPIIO6/GPIO35/FSPID/SUBSPID)
- net SLOT_A_DET: now also C6.1, R10.1, J2.14 (Pin_14), U1.6
- net SLOT_B_DET: now reaches U2.29 (SPIIO7/GPIO36/FSPICLK/SUBSPICLK)
- net SLOT_B_DET: now also J3.14 (Pin_14)
- net GPIO_37: now reaches U2.30 (SPIDQS/GPIO37/FSPIQ/SUBSPIQ)
- net MC_SD_1: now reaches U2.32 (MTCK/GPIO39/CLK_OUT3/SUBSPICS1)
- net MC_SD_2: now reaches U2.33 (MTDO/GPIO40/CLK_OUT2)
- net MC_DD_1: now reaches U2.34 (MTDI/GPIO41/CLK_OUT1)
- net MC_DD_2: now reaches U2.35 (MTMS/GPIO42)
- net ADC_BAT_EN renamed BZ_A_2
- net BZ_A_2: now also U3.15 (AIN2); no longer C3.1
- net ADC_VREF_EN renamed BZ_A_1
- net BZ_A_1: now also U3.16 (AIN1); no longer R12.2
- net GPIO11 renamed GPIO35
- net GPIO12 renamed GPIO36
- net GPIO13 renamed GPIO37
- new net: R20.1, U3.7 (BOUT1)
- new net: D2.1 (K), R12.1
- new net: D9.1 (K), R13.2
- new net: C9.1, U3.11 (VCP)
- new net: C10.2, U3.14 (VINT)
- new net: R14.1, U3.2 (AOUT1)
- new net BUZZER_A_+: R14.2
- new net BUZZER_A_-: U3.4 (AOUT2)
- new net BUZZER_B_+: R20.2
- new net BUZZER_B_-: U3.5 (BOUT2)
- new net MUX_1: J2.7 (Pin_7), J3.7 (Pin_7)
- new net MUX_2: J2.8 (Pin_8), J3.8 (Pin_8)
- new net MUX_3: J2.9 (Pin_9), J3.9 (Pin_9)
- new net SW3: J2.13 (Pin_13), J3.13 (Pin_13)
- new net VBUS_DET: R30.1, R6.2, U2.39 (GPIO1/TOUCH1/ADC1_CH0)
Other:
- note added: "Display Detection + MOSI Path"
- note added: "Slot A (Bottom)"
- note added: "Slot B (Top)"
- note added: "close to mcu mosi"
- note added: "this should be close to mcu"
- note removed: "A _|_ B"
- note removed: "Bat level reference"
- note removed: "TCL Order"
- note removed: "don't forget to route ldo_ctrl"
- moved on the sheet: BOOT1, C18, C3, C4, C5, D1, D10, D11, D3, D8, P11, P12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

Commit message: updated main board schematic
Parts:
- removed 1V1, 2.5V1: TestPoint_Alt, TestPoint:TestPoint_Pad_D1.5mm, symbol Connector:TestPoint_Alt
- removed D3, D9: LED, LED_SMD:LED_0603_1608Metric_Pad1.05x0.95mm_HandSolder, symbol Device:LED
- removed R9: 2.2K, Resistor_SMD:R_0603_1608Metric_Pad0.98x0.95mm_HandSolder, symbol Device:R
- added C21, C3: 1nF, Capacitor_SMD:C_0603_1608Metric_Pad1.08x0.95mm_HandSolder, symbol Device:C
- added C22: 0.1uF, Capacitor_SMD:C_0805_2012Metric_Pad1.18x1.45mm_HandSolder, symbol Device:C
- added D1: LED, LED_SMD:LED_0603_1608Metric_Pad1.05x0.95mm_HandSolder, symbol Device:LED
- added J3, J4, J5: Conn_01x02_Pin, symbol Connector:Conn_01x02_Pin
- added R15, R16: 4.7k, Resistor_SMD:R_0603_1608Metric_Pad0.98x0.95mm_HandSolder, symbol Device:R
- added RESET2: SW_Push, Luis:Button_3x4x2.5, symbol Switch:SW_Push
- added U4: DS3231MZ, Package_SO:SOIC-8_3.9x4.9mm_P1.27mm, symbol Timer_RTC:DS3231MZ
- added U8: 74LVC1G3157, symbol 74xGxx:74LVC1G3157
- C1: value 1uF -> 100nF
- C5: renamed from C9; footprint Capacitor_SMD:C_0805_2012Metric_Pad1.18x1.45mm_HandSolder -> Capacitor_SMD:C_0603_1608Metric_Pad1.08x0.95mm_HandSolder
- C8: renamed from C6; footprint (none) -> Capacitor_SMD:C_0603_1608Metric_Pad1.08x0.95mm_HandSolder
- J1: renamed from J2; footprint (none) -> Connector_PinHeader_1.27mm:PinHeader_2x12_P1.27mm_Vertical
- J2: renamed from J3; footprint (none) -> Connector_PinHeader_1.27mm:PinHeader_2x12_P1.27mm_Vertical
- R10: value 10k -> 2.2K
- R11: renamed from R14; footprint (none) -> Resistor_SMD:R_0603_1608Metric_Pad0.98x0.95mm_HandSolder
- R12: renamed from R20; footprint (none) -> Resistor_SMD:R_0603_1608Metric_Pad0.98x0.95mm_HandSolder
- R21: renamed from R3; value 1M -> 100k
- R22: renamed from R4; value 1M -> 100k
- R9: renamed from R13; value 2.2K -> 100k
- U3: renamed from U1; footprint (none) -> Package_TO_SOT_SMD:SOT-23-6_Handsoldering
- renumbered C13 to C11, C14 to C12, C3 to C13, C15 to C14, C16 to C15, C17 to C16, C7 to C17, C4 to C19, C5 to C20, C10 to C4, C11 to C6, C12 to C7, C8 to C9, D1 to D2, D2 to D3, D6 to D4, D7 to D5, D10 to D6, D8 to D7, D11 to D8, J1 to J6, P11 to P1, P12 to P2, P13 to P3, P46 to P4, Q3 to Q1, Q4 to Q2, Q6 to Q3, Q7 to Q4, Q8 to Q6, Q9 to Q7, R2 to R1, R11 to R13, R12 to R14, R5 to R2, R24 to R23, R25 to R24, R26 to R25, R27 to R26, R6 to R27, R30 to R28, R28 to R29, R1 to R3, R29 to R30, R33 to R32, R32 to R33, R35 to R34, R7 to R4, R8 to R5, R19 to R6, R18 to R7, R17 to R8, U2 to U1, U3 to U2
Connections:
- net CTRL is gone; now on net SLOT_B_DET: U1.31 (GPIO38/FSPIWP/SUBSPIWP)
- net GPIO14 is gone; now on net VBUS_DET: U1.22 (GPIO14/TOUCH14/ADC2_CH3/FSPIWP/FSPIDQS/SUBSPIWP)
- net GPIO_10 is gone; now on net LDO_LATCH: U1.18 (GPIO10/TOUCH10/ADC1_CH9/FSPICS0/FSPIIO4/SUBSPICS0)
- net GPIO_21 is gone; now on net SLOT_A_DET: U1.23 (GPIO21)
- net GPIO_37 is gone; now on net VCC_CTRL_EN: U1.30 (SPIDQS/GPIO37/FSPIQ/SUBSPIQ)
- net MC_DD_1 is gone; now on net MUX_3: U1.34 (MTDI/GPIO41/CLK_OUT1)
- net MC_SD_1 is gone; now on net MUX_1: U1.32 (MTCK/GPIO39/CLK_OUT3/SUBSPICS1)
- net MC_SD_2 is gone; now on net MUX_2: U1.33 (MTDO/GPIO40/CLK_OUT2)
- net SW2 is gone; now on net SW_2: J1.12 (Pin_12), J2.12 (Pin_12)
- net SW3 is gone; now on net SW_3: J1.13 (Pin_13), J2.13 (Pin_13)
- net ADC_BAT: now also U1.7 (GPIO7/TOUCH7/ADC1_CH6)
- net BLANK: no longer U1.9 (GPIO16/U0CTS/ADC2_CH5/XTAL_32K_N)
- net BUZZER_A_+: now also J3.1 (Pin_1)
- net BUZZER_A_-: now also J3.2 (Pin_2)
- net BUZZER_B_+: now also J4.1 (Pin_1)
- net BUZZER_B_-: now also J4.2 (Pin_2)
- net GND: now also R9.2, C21.2, C22.1, C3.1, J5.2 (Pin_2), RESET2.1, U4.5 (GND), U8.2 (GND); no longer J1.10 (Pin_10), J2.10 (Pin_10), R9.1
- net LDO: now also R15.2, R16.2, U4.6 (VBAT)
- net LDO_CTRL: now also C22.2, U8.5 (VCC); no longer R10.2, U2.1 (~{SLEEP})
- net LDO_CTRL_EN: now also U1.29 (SPIIO7/GPIO36/FSPICLK/SUBSPICLK); no longer U1.12 (GPIO8/TOUCH8/ADC1_CH7/SUBSPICS1)
- net LDO_LATCH: no longer U1.7 (GPIO7/TOUCH7/ADC1_CH6)
- net MISO(SOUT): now also U8.4
- net SLOT_A_DET: no longer R10.1, U1.28 (SPIIO6/GPIO35/FSPID/SUBSPID)
- net SLOT_B_DET: now also C21.1, U8.6; no longer U1.29 (SPIIO7/GPIO36/FSPICLK/SUBSPICLK)
- net SOUT_A: now also U8.1
- net SOUT_B: now also U8.3
- net VBUS_DET: no longer U1.39 (GPIO1/TOUCH1/ADC1_CH0)
- net VCC_CTRL: now also R10.1
- net VCC_CTRL_EN: no longer U1.17 (GPIO9/TOUCH9/ADC1_CH8/FSPIHD/SUBSPIHD)
- net at U2.8 (~{FAULT}): now also D1.1 (K)
- net RTC_~{INT}: now reaches U1.16 (GPIO46)
- net RTC_~{INT}: now also R9.1, U4.3 (~{INT}/SQW)
- net at U1.8 (GPIO15/U0RTS/ADC2_CH4/XTAL_32K_P): now also C3.2
- net SW_3: now reaches U1.15 (GPIO3/TOUCH3/ADC1_CH2)
- net ADC_BAT_V renamed SW_2
- net GPIO35: no longer names the net of P1.1
- net GPIO36: no longer names the net of P2.1
- net GPIO37: no longer names the net of P3.1
- net GPIO46: no longer names the net of P4.1
- net MC_DD_2 renamed MUX_4
- net MUX_4: now also J1.10 (Pin_10), J2.10 (Pin_10)
- net SW1 renamed SW_1
- net SW_1: now also U1.39 (GPIO1/TOUCH1/ADC1_CH0); no longer D2.C, D7.C
- new net: RESET2.2, U4.4 (~{RST})
- new net: D1.2 (A), R10.2
- new net DRV_~{SLEEP}: U1.28 (SPIIO6/GPIO35/FSPID/SUBSPID), U2.1 (~{SLEEP})
- new net RTC_BAT_+: J5.1 (Pin_1), U4.2 (VCC)
- new net RTC_CLK: U1.9 (GPIO16/U0CTS/ADC2_CH5/XTAL_32K_N), U4.1 (32KHZ)
- new net RTC_SCL: R16.1, U1.17 (GPIO9/TOUCH9/ADC1_CH8/FSPIHD/SUBSPIHD), U4.8 (SCL)
- new net RTC_SDA: R15.1, U1.12 (GPIO8/TOUCH8/ADC1_CH7/SUBSPICS1), U4.7 (SDA)
- new net SW_PWR: D2.C, D7.C
Other:
- note added: "Audio Circuit -> 2 Full H Bridge"
- note added: "Display Detection + MOSI and MISO Path"
- note added: "Enable Circuit"
- note added: "RTC"
- note added: "USB-C"
- note removed: "Display Detection + MOSI Path"
- note removed: "Enable reset circuit"
- note removed: "Signal Selection"
- moved on the sheet: BOOT1, C1, C19, C2, C20, C4, C5, C6, C7, C8, C9, D2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

Commit message: added docs and v2 of the main pcb is about done
Parts:
- removed C2: 0.1uF, Capacitor_SMD:C_0805_2012Metric_Pad1.18x1.45mm_HandSolder, symbol Device:C
- removed D2, D7, D8: BAT20J, BAT20JFILM:SOD-323, symbol BAT20JFILM:BAT20JFILM
- removed D6: BAT20JFILM, BAT20JFILM:SOD-323, symbol BAT20JFILM:BAT20JFILM
- removed P1, P2, P3, P4, RX1: TestPoint_Alt, TestPoint:TestPoint_Pad_D1.5mm, symbol Connector:TestPoint_Alt
- removed R2: 0, Resistor_SMD:R_0603_1608Metric_Pad0.98x0.95mm_HandSolder, symbol Device:R
- added C21: 100nF, Capacitor_SMD:C_0805_2012Metric_Pad1.18x1.45mm_HandSolder, symbol Device:C
- added D2, D6, D7, D8: BAT20J, Diode_SMD:D_SOD-323_HandSoldering, symbol Diode:BAT48JFILM
- added PWR1: SW_Push, Luis:Kahil Mute 6.2x6.2x7.3, symbol Switch:SW_Push
- added R30: 10k, Resistor_SMD:R_0603_1608Metric_Pad0.98x0.95mm_HandSolder, symbol Device:R
- BUZZER A1: renamed from J3; footprint (none) -> Connector_JST:JST_XH_B2B-XH-A_1x02_P2.50mm_Vertical
- BUZZER B1: renamed from J4; footprint (none) -> Connector_JST:JST_XH_B2B-XH-A_1x02_P2.50mm_Vertical
- CELL1: renamed from J5; footprint (none) -> Connector_PinHeader_1.27mm:PinHeader_1x02_P1.27mm_Vertical
- U4: renamed from U8; footprint (none) -> Package_TO_SOT_SMD:SOT-23-6_Handsoldering
- renumbered LDO1 to 3v3, J1 to A1, J2 to B1, U7 to BMS1, C9 to C10, C3 to C2, C4 to C3, C5 to C4, C6 to C5, C7 to C6, C8 to C7, C22 to C8, C21 to C9, U2 to DRV1, GND2 to G1, GND3 to GND2, GND4 to GND3, GND5 to GND4, LDO_1 to LDO1, R11 to R10, R12 to R11, R13 to R12, R14 to R13, R15 to R14, R16 to R15, R21 to R16, R22 to R17, R23 to R18, R24 to R19, R3 to R2, R25 to R20, R26 to R21, R27 to R22, R28 to R23, R29 to R24, R30 to R25, R31 to R26, R32 to R27, R33 to R28, R34 to R29, R4 to R3, R5 to R4, R6 to R5, R7 to R6, R8 to R7, R9 to R8, R10 to R9, RESET1 to RST1, U4 to RTC1, RESET2 to RTC_RST1, U6 to TP4056, U5 to U6, VCC_1 to VCC2
Connections:
- net BLANK: now also A1.17 (Pin_17), B1.17 (Pin_17), U1.21 (GPIO13/TOUCH13/ADC2_CH2/FSPIQ/FSPIIO7/SUBSPIQ); no longer A1.18 (Pin_18), B1.18 (Pin_18)
- net BUZZER_A_+: now also DRV1.2 (AOUT1); no longer R10.2
- net BUZZER_A_-: now also R10.2; no longer DRV1.4 (AOUT2)
- net BUZZER_B_+: now also DRV1.7 (BOUT1); no longer R11.2
- net BUZZER_B_-: now also R11.2; no longer DRV1.5 (BOUT2)
- net BZ_A_1: now also U1.5 (GPIO5/TOUCH5/ADC1_CH4); no longer U1.4 (GPIO4/TOUCH4/ADC1_CH3)
- net BZ_A_2: now also U1.4 (GPIO4/TOUCH4/ADC1_CH3); no longer U1.5 (GPIO5/TOUCH5/ADC1_CH4)
- net EN: now also RST1.1
- net GND: now also C21.2, PWR1.2; no longer A1.15 (Pin_15), A1.16 (Pin_16), B1.15 (Pin_15), B1.16 (Pin_16)
- net SLOT_A_DET: now also C9.1, U4.6
- net SLOT_B_DET: no longer C9.1, U4.6
- net SW_PWR: now also C21.1, D2.1 (K), D7.1 (K), PWR1.1, R30.2
- net VBUS: now also D6.2 (A), D8.2 (A)
- net VCC: now also D6.1 (K), R30.1
- net at R11.1: now also DRV1.5 (BOUT2); no longer DRV1.7 (BOUT1)
- net at C17.2, Q4.3 (D), Q6.1 (G)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: now also D7.2 (A)
- net at Q4.1 (G), Q7.2 (S), R27.1: now also D8.1 (K)
- net at R10.1: now also DRV1.4 (AOUT2); no longer DRV1.2 (AOUT1)
- net at U1.6 (GPIO6/TOUCH6/ADC1_CH5): now also D2.2 (A)
- net MISO(SOUT) renamed DCSIN_B
- net DCSIN_B: now also B1.18 (Pin_18); no longer U1.21 (GPIO13/TOUCH13/ADC2_CH2/FSPIQ/FSPIIO7/SUBSPIQ)
- net MOSI(SIN) renamed GSSIN
- net SIN_B renamed GSSIN_B
- removed net SOUT_A: A1.17 (Pin_17), U3.3, U4.1
- net SOUT_B renamed DCSOUT_A
- net DCSOUT_A: now also A1.16 (Pin_16); no longer B1.17 (Pin_17)
- net U0RXD renamed DCSIN
- net DCSIN: now also A1.18 (Pin_18), U4.1
- net XLAT renamed GSLAT
- new net GSSOUT_A: A1.15 (Pin_15), U3.3
- no-connect marks 2 -> 6
Other:
- note added: "Display Detection + GSSIN and DCSIN Path"
- note removed: "Display Detection + MOSI and MISO Path"
- note removed: "GPIO (Extra)"
- moved on the sheet: C1, C9, R1, R10, R11, R5, R6, R7, RST1, TX1, U4A

Commit message: v2.0 of the main and display board is ready and in production
Parts:
- added 3v32: TestPoint_Alt, TestPoint:TestPoint_Pad_D1.5mm, symbol Connector:TestPoint_Alt
- renumbered 3v3 to 3v31, C21 to C1, C9 to C10, C10 to C11, C11 to C12, C12 to C13, C13 to C14, C14 to C15, C15 to C16, C16 to C17, C17 to C18, C18 to C19, C1 to C2, C19 to C20, C20 to C21, C2 to C3, C3 to C4, C4 to C5, C5 to C6, C6 to C7, C7 to C8, C8 to C9, GND6 to GND5, GND7 to GND6, J6 to J1, R30 to R1, R9 to R10, R10 to R11, R11 to R12, R12 to R13, R13 to R14, R14 to R15, R15 to R16, R16 to R17, R17 to R18, R18 to R19, R1 to R2, R19 to R20, R20 to R21, R21 to R22, R22 to R23, R23 to R24, R24 to R25, R25 to R26, R26 to R27, R27 to R28, R28 to R29, R2 to R3, R29 to R30, R3 to R4, R4 to R5, R5 to R6, R6 to R7, R7 to R8, R8 to R9, TP4056 to TP1, U3 to U2, U4 to U3, U6 to U4
Connections:
- net LDO: now also 3v32.1
Other:
- moved on the sheet: 3v31, LDO1, VCC2

Commit message: detected wrong connections in the rtc module
Parts:
- R11: value 300 -> 110
- R26: value R -> 1.5k
Changed lines of the file:
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@@
 			)
 		)
-		(property "Value" "R"
+		(property "Value" "1.5k"
 			(at 387.35 76.2 0)
 			(effects
@@
 			)
 		)
-		(property "Value" "300"
+		(property "Value" "110"
 			(at 158.75 57.15 90)
 			(effects

Commit message: new version in the works, time is not yet functional but the new board is very much working
ds3231 vbat is switched with the vcc - fixed
have to fix capacitor resonance since it is really annoying
Parts:
- added C22: 0.1uF, Capacitor_SMD:C_0805_2012Metric_Pad1.18x1.45mm_HandSolder, symbol Device:C
Connections:
- net GND: now also C22.1
- net LDO: now also RTC1.2 (VCC), C22.2; no longer RTC1.6 (VBAT)
- net RTC_BAT_+: now also RTC1.6 (VBAT); no longer RTC1.2 (VCC)
Other:
- moved on the sheet: CELL1

Commit message: refined screens in v2.0, usb detection and sleep modes, some tweaks in the spi transmission solves brightness switching, esp now disabled for now since the peak currents sometimes reset the led driver
also matched the netscore online demo's logic to the currently being used on the devices, developed new 3d models for the new boards
Parts:
- D3: value LED -> BLUE
- D4: value LED -> orange
- D5: value LED -> green
- R12: value 300 -> 110
Connections:
- net LDO: now also RTC1.6 (VBAT); no longer RTC1.2 (VCC)
- net RTC_BAT_+: now also RTC1.2 (VCC); no longer RTC1.6 (VBAT)
Other:
- moved on the sheet: C3
Changed lines of the file:
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@@
 	)
 	(junction
+		(at 218.44 35.56)
+		(diameter 0)
+		(color 0 0 0 0)
+	)
+	(junction
 		(at 245.11 146.05)
 		(diameter 0)
@@
 	)
 	(junction
-		(at 218.44 35.56)
-		(diameter 0)
-		(color 0 0 0 0)
-	)
-	(junction
 		(at 384.81 81.28)
 		(diameter 0)
@@
 	(wire
 		(pts
+			(xy 232.41 35.56) (xy 218.44 35.56)
+		)
+		(stroke
+			(width 0)
+			(type default)
+		)
+	)
+	(wire
+		(pts
 			(xy 431.8 190.5) (xy 443.23 190.5)
 		)
@@
 	(wire
 		(pts
-			(xy 21.59 120.65) (xy 21.59 118.11)
-		)
-		(stroke
-			(width 0)
-			(type default)
-		)
-	)
-	(wire
-		(pts
 			(xy 134.62 110.49) (xy 134.62 105.41)
 		)
@@
 	(wire
 		(pts
-			(xy 218.44 35.56) (xy 234.95 35.56)
-		)
-		(stroke
-			(width 0)
-			(type default)
-		)
-	)
-	(wire
-		(pts
 			(xy 182.88 125.73) (xy 182.88 129.54)
 		)
@@
 	(wire
 		(pts
-			(xy 34.29 120.65) (xy 39.37 120.65)
-		)
-		(stroke
-			(width 0)
-			(type default)
-		)
-	)
-	(wire
-		(pts
 			(xy 137.16 123.19) (xy 140.97 123.19)
 		)
@@
 	(wire
 		(pts
+			(xy 21.59 118.11) (xy 39.37 118.11)
+		)
+		(stroke
+			(width 0)
+			(type default)
+		)
+	)
+	(wire
+		(pts
 			(xy 313.69 116.84) (xy 313.69 120.65)
 		)
@@
 	(wire
 		(pts
-			(xy 238.76 40.64) (xy 232.41 40.64)
-		)
-		(stroke
-			(width 0)
-			(type default)
-		)
-	)
-	(wire
-		(pts
 			(xy 114.3 50.8) (xy 101.6 50.8)
 		)
@@
 	(wire
 		(pts
-			(xy 21.59 118.11) (xy 39.37 118.11)
-		)
-		(stroke
-			(width 0)
-			(type default)
-		)
-	)
-	(wire
-		(pts
 			(xy 113.03 33.02) (xy 140.97 33.02)
 		)
@@
 	(wire
 		(pts
-			(xy 21.59 128.27) (xy 21.59 132.08)
+			(xy 21.59 130.81) (xy 21.59 132.08)
 		)
 		(stroke
@@
 	(wire
 		(pts
+			(xy 34.29 120.65) (xy 39.37 120.65)
+		)
+		(stroke
+			(width 0)
+			(type default)
+		)
+	)
+	(wire
+		(pts
 			(xy 120.65 50.8) (xy 114.3 50.8)
 		)
@@
 	(wire
 		(pts
-			(xy 232.41 40.64) (xy 232.41 44.45)
+			(xy 232.41 35.56) (xy 232.41 44.45)
 		)
 		(stroke
@@
 	(wire
 		(pts
+			(xy 21.59 118.11) (xy 21.59 123.19)
+		)
+		(stroke
+			(width 0)
+			(type default)
+		)
+	)
+	(wire
+		(pts
 			(xy 331.47 203.2) (xy 336.55 203.2)
 		)
@@
 	)
 	(label "RTC_BAT_+"
-		(at 238.76 40.64 0)
+		(at 234.95 35.56 0)
 		(effects
 			(font
@@
 			)
 		)
-		(property "Value" "300"
+		(property "Value" "110"
 			(at 158.75 69.85 90)
 			(effects
@@
 			)
 		)
-		(property "Value" "LED"
+		(property "Value" "BLUE"
 			(at 165.1 167.64 0)
 			(effects
@@
 	(symbol
 		(lib_id "Device:C")
-		(at 21.59 124.46 0)
+		(at 21.59 127 0)
 		(mirror x)
 		(unit 1)
@@
 		(dnp no)
 		(property "Reference" "C3"
-			(at 18.034 123.952 0)
+			(at 18.034 126.492 0)
 			(effects
 				(font
@@
 		)
 		(property "Value" "1nF"
-			(at 18.796 126.238 0)
+			(at 18.796 128.778 0)
 			(effects
 				(font
@@
 		)
 		(property "Footprint" "Capacitor_SMD:C_0603_1608Metric_Pad1.08x0.95mm_HandSolder"
-			(at 22.5552 120.65 0)
+			(at 22.5552 123.19 0)
 			(effects
 				(font
@@
 		)
 		(property "Datasheet" "~"
-			(at 21.59 124.46 0)
+			(at 21.59 127 0)
 			(effects
 				(font
@@
 		)
 		(property "Description" "Unpolarized capacitor"
-			(at 21.59 124.46 0)
+			(at 21.59 127 0)
 			(effects
 				(font
@@
 			)
 		)
-		(property "Value" "LED"
+		(property "Value" "orange"
 			(at 347.98 62.23 0)
 			(effects
@@
 		)
 		(property "Value" "5.1K"
-			(at 64.516 35.56 90)
+			(at 64.516 35.306 90)
 			(effects
 				(font
@@
 		)
 		(property "Value" "5.1K"
-			(at 75.692 45.72 90)
+			(at 75.692 45.212 90)
 			(effects
 				(font
@@
 			)
 		)
-		(property "Value" "LED"
+		(property "Value" "green"
 			(at 347.98 76.2 0)
 			(effects
